File: node_v3_1/node_v3_1/node_v3_1.kicad_sch (KiCad schematic)
At the start: 65 parts, among them J1 Conn_Coaxial, J10 3V3OUT, J12 12402012E212A, J13 DBG, J14 VIN, J15 Conn_01x16_Pin, J2 Micro_SD_Card, J6 BAT, Q1 2N3904, SW1 PTS526, SW2 PTS526, U1 RFM69HCW, U2 MCP7940N-xSN, U3 MCP73831-2-OT, U4 ADP2108AUJ-3.3, U5 CAT3200-5, U6 RP2040, U7 W25Q128JVS, Y1 445C35A12M00000, Y2 SC32S-7PF20PPM

Commit message: v3.1 begin
Parts:
- removed J10: 3V3OUT, Connector_PinHeader_2.54mm:PinHeader_1x02_P2.54mm_Vertical, symbol Connector:Conn_01x02_Pin
- removed J12: 12402012E212A, custom:AMPHENOL_12402012E212A, symbol custom:12402012E212A
- removed J13: DBG, Connector_PinHeader_2.54mm:PinHeader_1x03_P2.54mm_Vertical, symbol Connector:Conn_01x03_Pin
- removed J14: VIN, Connector_PinHeader_2.54mm:PinHeader_1x02_P2.54mm_Vertical, symbol Connector:Conn_01x02_Pin
- removed J15: Conn_01x16_Pin, Connector_PinHeader_2.54mm:PinHeader_1x16_P2.54mm_Vertical, symbol Connector:Conn_01x16_Pin
- removed J2: Micro_SD_Card, Connector_Card:microSD_HC_Molex_104031-0811, symbol Connector:Micro_SD_Card
- removed J6: BAT, Connector_PinHeader_2.54mm:PinHeader_1x02_P2.54mm_Vertical, symbol Connector:Conn_01x02_Pin
- removed R14: R, Resistor_SMD:R_0805_2012Metric_Pad1.20x1.40mm_HandSolder, symbol Device:R
- removed U1: RFM69HCW, RF_Module:HOPERF_RFM9XW_SMD, symbol RF_Module:RFM69HCW
- removed U2: MCP7940N-xSN, Package_SO:SOIC-8_3.9x4.9mm_P1.27mm, symbol Timer_RTC:MCP7940N-xSN
- removed U3: MCP73831-2-OT, Package_TO_SOT_SMD:SOT-23-5, symbol Battery_Management:MCP73831-2-OT
- removed U4: ADP2108AUJ-3.3, Package_TO_SOT_SMD:TSOT-23-5, symbol Regulator_Switching:ADP2108AUJ-3.3
- removed U5: CAT3200-5, Package_TO_SOT_SMD:SOT-23-6, symbol Regulator_SwitchedCapacitor:CAT3200-5
- removed U6: RP2040, Package_DFN_QFN:QFN-56-1EP_7x7mm_P0.4mm_EP3.2x3.2mm, symbol MCU_RaspberryPi:RP2040
- removed U7: W25Q128JVS, Package_SO:SOIC-8_5.23x5.23mm_P1.27mm, symbol Memory_Flash:W25Q128JVS
- added J2: 12402012E212A, custom:AMPHENOL_12402012E212A, symbol custom:12402012E212A
- added J3: Micro_SD_Card, Connector_Card:microSD_HC_Molex_104031-0811, symbol Connector:Micro_SD_Card
- added J4: VIN, Connector_PinHeader_2.54mm:PinHeader_1x02_P2.54mm_Vertical, symbol Connector:Conn_01x02_Pin
- added J5: BAT, Connector_PinHeader_2.54mm:PinHeader_1x02_P2.54mm_Vertical, symbol Connector:Conn_01x02_Pin
- added J7: DBG, Connector_PinHeader_2.54mm:PinHeader_1x03_P2.54mm_Vertical, symbol Connector:Conn_01x03_Pin
- added J8: Conn_01x16_Pin, Connector_PinHeader_2.54mm:PinHeader_1x16_P2.54mm_Vertical, symbol Connector:Conn_01x16_Pin
- added U1: MCP73831-2-OT, Package_TO_SOT_SMD:SOT-23-5, symbol Battery_Management:MCP73831-2-OT
- added U2: W25Q128JVS, Package_SO:SOIC-8_5.23x5.23mm_P1.27mm, symbol Memory_Flash:W25Q128JVS
- added U3: ADP2108AUJ-3.3, Package_TO_SOT_SMD:TSOT-23-5, symbol Regulator_Switching:ADP2108AUJ-3.3
- added U4: RP2040, Package_DFN_QFN:QFN-56-1EP_7x7mm_P0.4mm_EP3.2x3.2mm, symbol MCU_RaspberryPi:RP2040
- added U5: RFM69HCW, RF_Module:HOPERF_RFM9XW_SMD, symbol RF_Module:RFM69HCW
- added U6: CAT3200-5, Package_TO_SOT_SMD:SOT-23-6, symbol Regulator_SwitchedCapacitor:CAT3200-5
- added U7: MCP7940N-xSN, Package_SO:SOIC-8_3.9x4.9mm_P1.27mm, symbol Timer_RTC:MCP7940N-xSN
- C1: value 0.1uF -> 4.7uF; footprint Capacitor_SMD:C_0402_1005Metric -> Capacitor_SMD:C_0805_2012Metric_Pad1.18x1.45mm_HandSolder
- C10: value 100n -> 10uF; footprint Capacitor_SMD:C_0402_1005Metric_Pad0.74x0.62mm_HandSolder -> Capacitor_SMD:C_0805_2012Metric_Pad1.18x1.45mm_HandSolder
- C12, C14: value 100n -> 1uF; footprint Capacitor_SMD:C_0402_1005Metric_Pad0.74x0.62mm_HandSolder -> Capacitor_SMD:C_0805_2012Metric_Pad1.18x1.45mm_HandSolder
- C16: value 1u -> 100n; footprint Capacitor_SMD:C_0805_2012Metric_Pad1.18x1.45mm_HandSolder -> Capacitor_SMD:C_0402_1005Metric_Pad0.74x0.62mm_HandSolder
- C17: value 100n -> 0.1uF; footprint Capacitor_SMD:C_0402_1005Metric_Pad0.74x0.62mm_HandSolder -> Capacitor_SMD:C_0402_1005Metric
- C19: value 1u -> 1uF
- C21: value 15p -> 100n
- C22: value 15p -> 1u; footprint Capacitor_SMD:C_0402_1005Metric_Pad0.74x0.62mm_HandSolder -> Capacitor_SMD:C_0805_2012Metric_Pad1.18x1.45mm_HandSolder
- C24: value .1u -> 10u; footprint Capacitor_SMD:C_0402_1005Metric -> Capacitor_SMD:C_0805_2012Metric_Pad1.18x1.45mm_HandSolder
- C25: value 10u -> .1u; footprint Capacitor_SMD:C_0805_2012Metric_Pad1.18x1.45mm_HandSolder -> Capacitor_SMD:C_0402_1005Metric
- C3: value 10uF -> 15p; footprint Capacitor_SMD:C_0805_2012Metric_Pad1.18x1.45mm_HandSolder -> Capacitor_SMD:C_0402_1005Metric_Pad0.74x0.62mm_HandSolder
- C4: value 4.7uF -> 15p; footprint Capacitor_SMD:C_0805_2012Metric_Pad1.18x1.45mm_HandSolder -> Capacitor_SMD:C_0402_1005Metric_Pad0.74x0.62mm_HandSolder
- C5: value 10uF -> 1u
- C6, C8: value 1uF -> 100n; footprint Capacitor_SMD:C_0805_2012Metric_Pad1.18x1.45mm_HandSolder -> Capacitor_SMD:C_0402_1005Metric_Pad0.74x0.62mm_HandSolder
- C7: value 1uF -> 10uF
- R1: value 10K -> 2K
- R10: value 1k -> 10K
- R11: value 0 -> 10K
- R12: value R -> 10K
- R13: value R -> 0
- R15: value R -> 1K
- R2: value 470K -> 1k
- R3: value 470K -> 470
- R4: value 2K -> DNF
- R5: value 470 -> 27.4
- R6: value 1K -> 27.4
- R7: value 27.4 -> 10K
- R8: value 27.4 -> 470K
- R9: value DNF -> 470K
Connections:
- net 1V1: now also C5.1, C6.1, C9.1, U4.23 (DVDD), U4.45 (VREG_VOUT), U4.50 (DVDD); no longer C17.1, C18.1, C19.1
- net 3V3: now also C17.1, C18.1, C21.1, C22.1, C8.1, R10.1, R11.1, R4.1, J3.4 (VDD), J8.2 (Pin_2), U2.8 (VCC), U3.4 (FB), U4.1 (IOVDD), U4.10 (IOVDD), U4.22 (IOVDD), U4.33 (IOVDD), U4.42 (IOVDD), U4.43 (ADC_AVDD), U4.44 (VREG_IN), U4.48 (USB_VDD), U4.49 (IOVDD), U5.13 (3.3V), U7.8 (VCC); no longer C1.1, C12.1, C14.1, C5.1, C9.1, R13.1, R15.1, R9.1
- net 5V: now also C19.1, U6.1 (VOUT); no longer C8.1
- net 5V_CTRL: now also R7.2, U6.3 (~{SHDN}); no longer R1.2
- net 5V_OUT: now also J8.3 (Pin_3)
- net 5V_SW: now also R15.1, U4.4 (GPIO2); no longer R6.1
- net ANT: now also U5.9 (ANT)
- net BAT: now also C12.1, C2.1, C7.1, R8.1, J5.2 (Pin_2), U1.3 (V_{BAT}), U3.1 (Vin), U3.3 (EN), U6.5 (VIN); no longer C3.1, C4.1, C6.1, R2.1, R5.2
- net EXT_SW1: now also J8.16 (Pin_16), U4.15 (GPIO12)
- net EXT_SW2: now also J8.15 (Pin_15), U4.16 (GPIO13)
- net GND: now also C21.2, C22.2, C3.1, C4.1, C7.2, R1.2, R13.2, R9.2, J2.A1_B12 (GND), J2.B1_A12 (GND__1), J3.6 (VSS), J3.9 (SHIELD), J4.1 (Pin_1), J5.1 (Pin_1), J7.1 (Pin_1), J8.1 (Pin_1), U1.2 (V_{SS}), U2.4 (GND), U3.2 (GND), U4.19 (TESTEN), U4.57 (GND), U5.1 (GND), U5.10 (GND), U5.8 (GND), U6.2 (GND), U7.4 (VSS); no longer C14.2, C21.1, C22.1, C3.2, C4.2, R11.2, R3.2, R4.2
- net GP26: now also J8.13 (Pin_13), U4.38 (GPIO26_ADC0)
- net GP27: now also J8.12 (Pin_12), U4.39 (GPIO27_ADC1)
- net GP6: now also J8.14 (Pin_14), U4.8 (GPIO6)
- net I2C_SCK: now also J8.6 (Pin_6), U4.7 (GPIO5), U7.6 (SCL)
- net I2C_SDA: now also J8.7 (Pin_7), U4.6 (GPIO4), U7.5 (SDA)
- net MISO: now also R11.2, J3.7 (DAT0), J8.11 (Pin_11), U4.27 (GPIO16), U5.2 (MISO); no longer R13.2
- net MOSI: now also J3.3 (CMD), J8.10 (Pin_10), U4.30 (GPIO19), U5.3 (MOSI)
- net QSPI_CLK: now also U2.6 (CLK), U4.52 (QSPI_SCLK)
- net QSPI_CS: now also R2.2, R4.2, U2.1 (~{CS}), U4.56 (QSPI_SS); no longer R10.2, R9.2
- net QSPI_SD0: now also U2.5 (DI(IO0)), U4.53 (QSPI_SD0)
- net QSPI_SD1: now also U2.2 (DO(IO1)), U4.55 (QSPI_SD1)
- net QSPI_SD2: now also U2.3 (IO2), U4.54 (QSPI_SD2)
- net QSPI_SD3: now also U2.7 (IO3), U4.51 (QSPI_SD3)
- net RFM_CS: now also U4.28 (GPIO17), U5.5 (NSS)
- net RFM_RST: now also U4.31 (GPIO20), U5.6 (RESET)
- net RTC_MFP: now also U4.18 (GPIO15), U7.7 (MFP)
- net SD_CS: now also R12.2, J3.2 (DAT3/CD), U4.32 (GPIO21)
- net SPI_CS: now also J8.8 (Pin_8), U4.34 (GPIO22)
- net SPI_SCK: now also J3.5 (CLK), J8.9 (Pin_9), U4.29 (GPIO18), U5.4 (SCK)
- net SWD: now also J7.3 (Pin_3), U4.25 (SWD)
- net SWDCLK: now also J7.2 (Pin_2), U4.24 (SWCLK)
- net UART_RX: now also J8.4 (Pin_4), U4.3 (GPIO1)
- net UART_TX: now also J8.5 (Pin_5), U4.2 (GPIO0)
- net USB+: now also R5.1, J2.A6 (D+_A), J2.B6 (D+_B); no longer R7.1
- net USB-: now also R6.1, J2.A7 (D-_A), J2.B7 (D-_B); no longer R8.1
- net VIN: now also C1.1, J2.A4_B9 (VBUS), J2.B4_A9 (VBUS__1), J4.2 (Pin_2), U1.4 (V_{DD}); no longer C2.1
- net at D1.1 (K): now also R3.1; no longer R5.1
- net at SW1.3, SW1.4: now also R2.1; no longer R10.1
- net at R1.1: now also U1.5 (PROG)
- net at C26.1, Y2.1: now also U7.1 (X1)
- net at C27.1, Y2.2: now also U7.2 (X2)
- net at Y1.2: now also C3.2, U4.20 (XIN); no longer C21.2
- net at BT1.1 (+): now also U7.3 (VBAT)
- net at R8.2: now also R9.1, U4.40 (GPIO28_ADC2)
- net at R6.2: now also U4.46 (USB_DM); no longer Q1.2 (B)
- net at R15.2: now also Q1.2 (B)
- net at L1.1: now also U3.5 (SW)
- net at Y1.1: now also C4.2, U4.21 (XOUT); no longer C22.2
- net at SW2.3, SW2.4: now also U4.26 (RUN)
- new net: R7.1, U4.14 (GPIO11)
- new net: R5.2, U4.47 (USB_DP)
- new net: R3.2, U1.1 (STAT)
- new net: J3.1 (DAT2), R10.2
- new net: J2.SH1 (SHIELD), J2.SH2 (SHIELD__1), J2.SH3 (SHIELD__2), J2.SH4 (SHIELD__3), R13.1
- new net: C14.2, U6.4 (CNEG)
- new net: C14.1, U6.6 (CPOS)
- no-connect marks 0 -> 21
Other:
- note removed: "3V3 OUT"
