File: node_v3_1/node_v3_1/node_v3_1.kicad_sch (KiCad schematic)
At the start: 63 parts, among them J1 Conn_Coaxial, J2 12402012E212A, J3 Micro_SD_Card, J4 VIN, J5 BAT, J7 DBG, J8 Conn_01x16_Pin, Q1 2N3904, SW1 PTS526, SW2 PTS526, U1 MCP73831-2-OT, U2 W25Q128JVS, U3 ADP2108AUJ-3.3, U4 RP2040, U5 RFM69HCW, U6 CAT3200-5, U7 MCP7940N-xSN, Y1 445C35A12M00000, Y2 SC32S-7PF20PPM

Commit message: started pcb
Parts:
- removed C1, C2: 4.7uF, Capacitor_SMD:C_0805_2012Metric_Pad1.18x1.45mm_HandSolder, symbol Device:C
- removed D1: LED, LED_SMD:LED_1206_3216Metric_Pad1.42x1.75mm_HandSolder, symbol Device:LED
- removed J2: 12402012E212A, custom:AMPHENOL_12402012E212A, symbol custom:12402012E212A
- removed Q1: 2N3904, Package_TO_SOT_SMD:SC-59_Handsoldering, symbol PCM_Transistor_BJT_AKL:2N3904
- removed R3: 470, Resistor_SMD:R_0805_2012Metric_Pad1.20x1.40mm_HandSolder, symbol Device:R
- removed SW1, SW2: PTS526, custom:PTS526, symbol custom:PTS526
- removed U1: MCP73831-2-OT, Package_TO_SOT_SMD:SOT-23-5, symbol Battery_Management:MCP73831-2-OT
- added C28, C29: 4.7uF, Capacitor_SMD:C_0805_2012Metric_Pad1.18x1.45mm_HandSolder, symbol Device:C
- added D2: LED, LED_SMD:LED_1206_3216Metric_Pad1.42x1.75mm_HandSolder, symbol Device:LED
- added H1, H2, H3, H4: MountingHole, MountingHole:MountingHole_2.2mm_M2_Pad_Via, symbol Mechanical:MountingHole
- added J2: 12402012E212A, usbc:AMPHENOL_12402012E212A, symbol 12402012E212A:12402012E212A
- added Q1: 2N3904, Package_TO_SOT_SMD:SOT-23-3, symbol Transistor_BJT:2N3904
- added R14: 470, Resistor_SMD:R_0805_2012Metric_Pad1.20x1.40mm_HandSolder, symbol Device:R
- added U1: RST, pts526:SMT_FS, symbol 2024-05-28_14-35-54:PTS526_SK15_SMTR2_LFS
- added U8: MCP73831T-2ACI_OT, mcp73831:SOT95P280X145-5N, symbol MCP73831T-2ACI_OT:MCP73831T-2ACI_OT
- added U9: BOOTSEL, pts526:SMT_FS, symbol 2024-05-28_14-35-54:PTS526_SK15_SMTR2_LFS
- BT1: footprint custom:BAT-HLD-001-THM_TEC -> BAT-HLD-001:BAT_BAT-HLD-001-THM
- J1: footprint Connector_Coaxial:SMA_Samtec_SMA-J-P-X-ST-EM1_EdgeMount -> Connector_Coaxial:SMA_Samtec_SMA-J-P-H-ST-EM1_EdgeMount
- Y1: footprint kicad-footprints-master:XTAL_M445 -> custom:XTAL-445
- Y2: footprint custom:SC-32S -> sc32s:XTAL_SC32S-7PF20PPM_EPS
Connections:
- net 5V: now also Q1.3 (C)
- net 5V_OUT: now also Q1.1 (E)
- net BAT: now also C29.1, U8.3 (VBAT)
- net GND: now also R1.1, C28.2, C29.2, J2.A1_B12 (GND), J2.B1_A12 (GND__1), U1.1, U1.2, U8.2 (VSS), U9.1, U9.2; no longer C23.2, C25.2, R1.2
- net USB+: now also J2.A6 (D+_A), J2.B6 (D+_B)
- net USB-: now also J2.A7 (D-_A), J2.B7 (D-_B)
- net VIN: now also C28.1, D2.2 (A), J2.A4_B9 (VBUS), J2.B4_A9 (VBUS__1), U8.4 (VDD)
- net at U4.26 (RUN): now also U1.3, U1.4
- net at R15.2: now also Q1.2 (B)
- net at R13.1: now also J2.SH1 (SHIELD), J2.SH2 (SHIELD__1), J2.SH3 (SHIELD__2), J2.SH4 (SHIELD__3)
- net at R2.1: now also U9.3, U9.4
- new net: C23.2, C25.2
- new net: D2.1 (K), R14.1
- new net: R1.2, U8.5 (PROG)
- new net: R14.2, U8.1 (STAT)
Other:
- moved on the sheet: BT1, C10, C17, C24, C26, C27, C7, C8, L1, R13, R2, R4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

Commit message: ready to order(probably)
Parts:
- removed H1, H2, H3, H4: MountingHole, MountingHole:MountingHole_2.2mm_M2_Pad_Via, symbol Mechanical:MountingHole
- added H1, H2, H3, H4: MountingHole_Pad, MountingHole:MountingHole_2.2mm_M2_Pad, symbol Mechanical:MountingHole_Pad
- added R16, R3: 10K, Resistor_SMD:R_0805_2012Metric_Pad1.20x1.40mm_HandSolder, symbol Device:R
Connections:
- net 3V3: now also R16.1, R3.1
- net GND: now also C23.2, C25.2, H1.1, H2.1, H3.1, H4.1
- net MOSI: now also R3.2
- net UART_RX: now also J8.5 (Pin_5); no longer J8.4 (Pin_4)
- net UART_TX: now also J8.4 (Pin_4); no longer J8.5 (Pin_5)
- net USB_-: now reaches R6.2, U4.46 (USB_DM)
- net USB_+: now reaches R5.2, U4.47 (USB_DP)
- net at J3.8 (DAT1): now also R16.2
- no-connect marks 21 -> 20

Commit message: updates
Parts:
- added R17: 1k, symbol Device:R
Connections:
- net at C4.2, Y1.1: now also R17.1; no longer U4.21 (XOUT)
- new net: R17.2, U4.21 (XOUT)
Other:
- moved on the sheet: C3, C4, Y1
Changed lines of the file:
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@@
 	)
 	(junction
-		(at 55.88 241.3)
+		(at 39.37 241.3)
 		(diameter 0)
 		(color 0 0 0 0)
@@
 	)
 	(junction
-		(at 72.39 241.3)
+		(at 55.88 231.14)
 		(diameter 0)
 		(color 0 0 0 0)
 	)
 	(junction
-		(at 72.39 231.14)
+		(at 250.19 248.92)
 		(diameter 0)
 		(color 0 0 0 0)
 	)
 	(junction
-		(at 250.19 248.92)
+		(at 46.99 123.19)
 		(diameter 0)
 		(color 0 0 0 0)
 	)
 	(junction
-		(at 46.99 123.19)
+		(at 21.59 279.4)
 		(diameter 0)
 		(color 0 0 0 0)
 	)
 	(junction
-		(at 21.59 279.4)
+		(at 55.88 241.3)
 		(diameter 0)
 		(color 0 0 0 0)
@@
 	(wire
 		(pts
-			(xy 72.39 240.03) (xy 72.39 241.3)
+			(xy 55.88 240.03) (xy 55.88 241.3)
 		)
 		(stroke
@@
 	(wire
 		(pts
-			(xy 72.39 232.41) (xy 72.39 231.14)
+			(xy 55.88 232.41) (xy 55.88 231.14)
 		)
 		(stroke
@@
 	(wire
 		(pts
-			(xy 72.39 231.14) (xy 86.36 231.14)
+			(xy 55.88 231.14) (xy 86.36 231.14)
 		)
 		(stroke
@@
 	(wire
 		(pts
+			(xy 73.66 241.3) (xy 86.36 241.3)
+		)
+		(stroke
+			(width 0)
+			(type default)
+		)
+	)
+	(wire
+		(pts
 			(xy 36.83 101.6) (xy 40.64 101.6)
 		)
@@
 	(wire
 		(pts
-			(xy 55.88 231.14) (xy 55.88 241.3)
+			(xy 39.37 231.14) (xy 39.37 241.3)
 		)
 		(stroke
@@
 	(wire
 		(pts
+			(xy 55.88 241.3) (xy 66.04 241.3)
+		)
+		(stroke
+			(width 0)
+			(type default)
+		)
+	)
+	(wire
+		(pts
 			(xy 246.38 226.06) (xy 246.38 229.87)
 		)
@@
 	(wire
 		(pts
-			(xy 60.96 231.14) (xy 55.88 231.14)
+			(xy 44.45 231.14) (xy 39.37 231.14)
 		)
 		(stroke
@@
 	(wire
 		(pts
-			(xy 55.88 241.3) (xy 60.96 241.3)
+			(xy 39.37 241.3) (xy 44.45 241.3)
 		)
 		(stroke
@@
 	(wire
 		(pts
-			(xy 55.88 241.3) (xy 55.88 243.84)
+			(xy 39.37 241.3) (xy 39.37 243.84)
 		)
 		(stroke
@@
 	(wire
 		(pts
-			(xy 72.39 241.3) (xy 86.36 241.3)
-		)
-		(stroke
-			(width 0)
-			(type default)
-		)
-	)
-	(wire
-		(pts
 			(xy 137.16 198.12) (xy 139.7 198.12)
 		)
@@
 	(wire
 		(pts
-			(xy 72.39 241.3) (xy 68.58 241.3)
+			(xy 55.88 241.3) (xy 52.07 241.3)
 		)
 		(stroke
@@
 	(wire
 		(pts
-			(xy 72.39 231.14) (xy 68.58 231.14)
+			(xy 55.88 231.14) (xy 52.07 231.14)
 		)
 		(stroke
@@
 	(symbol
 		(lib_id "Device:Crystal")
-		(at 72.39 236.22 90)
+		(at 55.88 236.22 90)
 		(unit 1)
 		(exclude_from_sim no)
@@
 		(on_board yes)
 		(dnp no)
-		(fields_autoplaced yes)
 		(property "Reference" "Y1"
-			(at 76.2 234.95 90)
+			(at 59.69 234.95 90)
 			(effects
 				(font
@@
 		)
 		(property "Value" "445C35A12M00000"
-			(at 76.2 237.49 90)
+			(at 59.69 237.49 90)
 			(effects
 				(font
@@
 		)
 		(property "Footprint" "custom:XTAL-445"
-			(at 72.39 236.22 0)
+			(at 55.88 236.22 0)
 			(effects
 				(font
@@
 		)
 		(property "Datasheet" "~"
-			(at 72.39 236.22 0)
+			(at 55.88 236.22 0)
 			(effects
 				(font
@@
 		)
 		(property "Description" ""
-			(at 72.39 236.22 0)
+			(at 55.88 236.22 0)
 			(effects
 				(font
@@
 		(lib_name "GND_2")
 		(lib_id "power:GND")
-		(at 55.88 243.84 0)
+		(at 39.37 243.84 0)
 		(unit 1)
 		(exclude_from_sim no)
@@
 		(fields_autoplaced yes)
 		(property "Reference" "#PWR023"
-			(at 55.88 250.19 0)
+			(at 39.37 250.19 0)
 			(effects
 				(font
@@
 		)
 		(property "Value" "GND"
-			(at 55.88 248.92 0)
+			(at 39.37 248.92 0)
 			(effects
 				(font
@@
 		)
 		(property "Footprint" ""
-			(at 55.88 243.84 0)
+			(at 39.37 243.84 0)
 			(effects
 				(font
@@
 		)
 		(property "Datasheet" ""
-			(at 55.88 243.84 0)
+			(at 39.37 243.84 0)
 			(effects
 				(font
@@
 		)
 		(property "Description" "Power symbol creates a global label with name \"GND\" , ground"
-			(at 55.88 243.84 0)
+			(at 39.37 243.84 0)
 			(effects
 				(font
@@
 	(symbol
 		(lib_id "Device:C")
-		(at 64.77 231.14 90)
+		(at 48.26 231.14 90)
 		(unit 1)
 		(exclude_from_sim no)
@@
 		(dnp no)
 		(property "Reference" "C3"
-			(at 64.77 227.33 90)
+			(at 48.26 227.33 90)
 			(effects
 				(font
@@
 		)
 		(property "Value" "15p"
-			(at 64.77 234.95 90)
+			(at 48.26 234.95 90)
 			(effects
 				(font
@@
 		)
 		(property "Footprint" "Capacitor_SMD:C_0402_1005Metric_Pad0.74x0.62mm_HandSolder"
-			(at 68.58 230.1748 0)
+			(at 52.07 230.1748 0)
 			(effects
 				(font
@@
 		)
 		(property "Datasheet" "~"
-			(at 64.77 231.14 0)
+			(at 48.26 231.14 0)
 			(effects
 				(font
@@
 		)
 		(property "Description" ""
-			(at 64.77 231.14 0)
+			(at 48.26 231.14 0)
 			(effects
 				(font
@@
 	)
 	(symbol
+		(lib_id "Device:R")
+		(at 69.85 241.3 90)
+		(unit 1)
+		(exclude_from_sim no)
+		(in_bom yes)
+		(on_board yes)
+		(dnp no)
+		(property "Reference" "R17"
+			(at 67.818 243.84 90)
+			(effects
+				(font
+					(size 1.27 1.27)
+				)
+			)
+		)
+		(property "Value" "1k"
+			(at 71.882 243.84 90)
+			(effects
+				(font
+					(size 1.27 1.27)
+				)
+			)
+		)
+		(property "Footprint" ""
+			(at 69.85 243.078 90)
+			(effects
+				(font
+					(size 1.27 1.27)
+				)
+				(hide yes)
+			)
+		)
+		(property "Datasheet" "~"
+			(at 69.85 241.3 0)
+			(effects
+				(font
+					(size 1.27 1.27)
+				)
+				(hide yes)
+			)
+		)
+		(property "Description" "Resistor"
+			(at 69.85 241.3 0)
+			(effects
+				(font
+					(size 1.27 1.27)
+				)
+				(hide yes)
+			)
+		)
+		(pin "2"
+		)
+		(pin "1"
+		)
+		(instances
+			(project ""
+				(path "/e774f05c-3d76-4c30-8e02-47afd946aaf5"
+					(reference "R17")
+					(unit 1)
+				)
+			)
+		)
+	)
+	(symbol
 		(lib_name "GND_2")
 		(lib_id "power:GND")
@@
 	(symbol
 		(lib_id "Device:C")
-		(at 64.77 241.3 90)
+		(at 48.26 241.3 90)
 		(unit 1)
 		(exclude_from_sim no)
@@
 		(dnp no)
 		(property "Reference" "C4"
-			(at 64.77 237.49 90)
+			(at 48.26 237.49 90)
 			(effects
 				(font
@@
 		)
 		(property "Value" "15p"
-			(at 64.77 245.11 90)
+			(at 48.26 245.11 90)
 			(effects
 				(font
@@
 		)
 		(property "Footprint" "Capacitor_SMD:C_0402_1005Metric_Pad0.74x0.62mm_HandSolder"
-			(at 68.58 240.3348 0)
+			(at 52.07 240.3348 0)
 			(effects
 				(font
@@
 		)
 		(property "Datasheet" "~"
-			(at 64.77 241.3 0)
+			(at 48.26 241.3 0)
 			(effects
 				(font
@@
 		)
 		(property "Description" ""
-			(at 64.77 241.3 0)
+			(at 48.26 241.3 0)
 			(effects
 				(font
