File: node_v3_1/node_v3_1/node_v3_1.kicad_pcb (KiCad board)
At the start: 2 copper layers, 45.7 x 76.2 mm, 67 parts, among them J1 Conn_Coaxial, J2 12402012E212A, J3 Micro_SD_Card, J4 VIN, J5 BAT, J7 DBG, J8 Conn_01x16_Pin, Q1 2N3904, U1 RST, U2 W25Q128JVS, U3 ADP2108, U4 RP2040, U5 RFM69HCW, U6 CAT3200-5, U7 MCP7940, U8 MCP73831, U9 BOOTSEL, Y1 XTAL-445, Y2 SC32S

Commit message: finished layout(probably)
Parts:
- moved C23 83.1 mm to (162.1, 109.5), turned to -90 degrees
- moved R8 73.6 mm to (145.8, 62.2), turned to -90 degrees
- moved C25 73.1 mm to (164.3, 109.7), turned to -90 degrees
- moved R9 73.1 mm to (145.8, 66.0), turned to -90 degrees
- moved R2 71.9 mm to (138.2, 61.0), turned to 180 degrees
- moved R11 71.0 mm to (156.2, 109.5), turned to -90 degrees
- moved R4 70.9 mm to (137.2, 64.3), turned to 90 degrees
- moved R12 69.0 mm to (158.5, 109.5), turned to -90 degrees
- moved R10 68.7 mm to (153.9, 109.5), turned to -90 degrees
- moved R13 66.3 mm to (136.7, 56.9), turned to 90 degrees
- moved R7 63.6 mm to (147.8, 89.9)
- moved C5 60.4 mm to (145.5, 71.9), turned to 90 degrees
- moved C6 53.1 mm to (147.3, 72.7), turned to 90 degrees
- moved C9 51.7 mm to (148.6, 72.7), turned to 90 degrees
- moved C24 45.0 mm to (134.6, 79.2), turned to -90 degrees
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Connections:
- BT1 pad P1: (no net) -> Net-(BT1-+)
- BT1 pad P2: (no net) -> Net-(BT1-+)
- BT1 pad P3: (no net) -> Net-(BT1-+)
Other:
- copper layers 2 -> 4

Commit message: ready to order(probably)
Parts:
- added G***: LOGO, logos:wisdom_logo_lineborder, B.Cu at (150.1, 65.5)
- added G***: LOGO, logos:cat, B.Cu at (150.1, 82.0)
- added LOGO: , logos:qrcode, B.Cu at (162.8, 105.7)
- added LOGO: , logos:github_qr, B.Cu at (162.6, 120.5)
- added R16: 10K, Resistor_SMD:R_0805_2012Metric_Pad1.20x1.40mm_HandSolder, F.Cu at (160.5, 109.5)
- added R3: 10K, Resistor_SMD:R_0805_2012Metric_Pad1.20x1.40mm_HandSolder, F.Cu at (158.5, 109.5)
- H1, H2, H3, H4: value MountingHole -> MountingHole_Pad; footprint MountingHole:MountingHole_2.2mm_M2_Pad_Via -> MountingHole:MountingHole_2.2mm_M2_Pad
- U3: value ADP2108 -> ADP2108AUJ-3.3
- U7: value MCP7940 -> MCP7940N-xSN
- U8: value MCP73831 -> MCP73831T-2ACI_OT
- Y1: value XTAL-445 -> 445C35A12M00000
- Y2: value SC32S -> SC32S-7PF20PPM
- moved C8 8.44 mm to (137.2, 62.7)
- moved R7 5.09 mm to (148.0, 95.0)
- moved C17 4.97 mm to (150.5, 108.5), turned to -90 degrees
- moved U3 3.83 mm to (158.3, 81.5)
- moved C10 3.83 mm to (158.2, 78.2)
- moved C7 3.83 mm to (162.3, 81.5)
- moved L1 3.83 mm to (153.7, 81.7)
- moved U5 3.73 mm to (140.3, 108.1)
- moved Y2 3.08 mm to (132.9, 84.1)
- moved C26 3.08 mm to (131.3, 88.1)
- moved C27 3.08 mm to (134.4, 88.1), turned to -90 degrees
- moved BT1 2.94 mm to (140.2, 107.7)
- moved R2 2.93 mm to (141.0, 61.7)
- moved U4 2.92 mm to (143.2, 79.5)
- moved C3 2.82 mm to (138.5, 86.4)
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Connections:
- net Net-(U4-USB_DM) renamed /USB_-
- net Net-(U4-USB_DP) renamed /USB_+
- C23 pad 2: Net-(C23-Pad2) -> GND
- C25 pad 2: Net-(C23-Pad2) -> GND
- H1 pad 1: (no net) -> GND
- H2 pad 1: (no net) -> GND
- H3 pad 1: (no net) -> GND
- H4 pad 1: (no net) -> GND
- J3 pad 8: unconnected-(J3-DAT1-Pad8) -> Net-(J3-DAT1)
- J8 pad 4: UART_RX -> UART_TX
- J8 pad 5: UART_TX -> UART_RX
Routing:
- net 3V3: track 0.00 -> 179.0 mm, vias 0 -> 4
- net MISO: track 0.00 -> 103.3 mm, vias 0 -> 4
- net MOSI: track 0.00 -> 99.0 mm, vias 0 -> 6
- net SPI_SCK: track 0.00 -> 96.8 mm, vias 0 -> 5
- net BAT: track 0.00 -> 82.0 mm
- net GP6: track 0.00 -> 53.8 mm, vias 0 -> 2
- net SD_CS: track 0.00 -> 53.6 mm, vias 0 -> 5
- net Net-(BT1-+): track 0.00 -> 53.0 mm
- net RFM_RST: track 0.00 -> 48.0 mm, vias 0 -> 4
- net EXT_SW1: track 0.00 -> 45.5 mm, vias 0 -> 2
- net EXT_SW2: track 0.00 -> 44.0 mm, vias 0 -> 1
- net VIN: track 0.00 -> 44.0 mm, vias 0 -> 2
- net I2C_SCK: track 0.00 -> 42.7 mm, vias 0 -> 2
- net GP26: track 0.00 -> 42.3 mm, vias 0 -> 3
- net I2C_SDA: track 0.00 -> 42.0 mm, vias 0 -> 2
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- added copper zone on B.Cu, net GND
- added copper zone on F.Cu, net GND
Other:
- board text added: "+"
- board text added: "0.1u"
- board text added: "10K"
- board text added: "10u"
- board text added: "10uF"
- board text added: "15p"
- board text added: "1K"
- board text added: "1k"
- board text added: "1u"
- board text added: "1uF"
- board text added: "27.4"
- board text added: "2K"
- board text added: "3904"
- board text added: "4.7uF"
- board text added: "470"
- board text added: "470K"
- board text added: "6p"
- board text added: "ADP2108"
- board text added: "ANT"
- board text added: "BAT"
- board text added: "BOOTSEL"
- board text added: "C22"
- board text added: "CAT3200"
- board text added: "CLK"
- board text added: "GND"
- board text added: "GND 3V3 5V TX RX SCK SDA CS SCK MOSI MISO GP27 GP26 GP6 GP13 GP12"
- board text added: "M445"
- board text added: "MCP73831"
- board text added: "MCP7940"
- board text added: "RESET"
- board text added: "SC32S"
- board text added: "SWD"
- board text added: "VIN"
- board text added: "W25Q128"
- board text added: "WiSDOM Github"
- board text added: "WiSDOM Node v3.1 June 2024 By Amelia Vlahogiannis"
- board text added: "Y1"
- board text added: "wisdomresearch.net"
- board text added: "x5"
