File: node_v4_0/node_v4_0/node_v4_0.kicad_sch (KiCad schematic)
At the start: 28 parts, among them J1 Conn_Coaxial, J2 Micro_SD_Card, J3 12402012E212A, J4 VIN, J5 BAT, J6 DBG, J7 Conn_01x16_Pin, U8 MCP7940N-xSN, U9 RFM69HCW, Y2 SC32S-7PF20PPM

Commit message: converted v4 to different format and started the schematic(from scratch again)
Parts:
- removed BT1: Battery_Cell, BAT-HLD-001:BAT_BAT-HLD-001-THM, symbol Device:Battery_Cell
- removed C19, C23: 10u, Capacitor_SMD:C_0805_2012Metric_Pad1.18x1.45mm_HandSolder, symbol Device:C
- removed C24, C25: 6p, Capacitor_SMD:C_0603_1608Metric_Pad1.08x0.95mm_HandSolder, symbol Device:C
- removed C26: .1u, Capacitor_SMD:C_0402_1005Metric, symbol Device:C
- removed C27: 0.1uF, Capacitor_SMD:C_0402_1005Metric, symbol Device:C
- removed H1, H2, H3, H4: MountingHole_Pad, MountingHole:MountingHole_2.2mm_M2_Pad, symbol Mechanical:MountingHole_Pad
- removed J1: Conn_Coaxial, Connector_Coaxial:SMA_Samtec_SMA-J-P-H-ST-EM1_EdgeMount, symbol Connector:Conn_Coaxial
- removed J2: Micro_SD_Card, Connector_Card:microSD_HC_Molex_104031-0811, symbol Connector:Micro_SD_Card
- removed J3: 12402012E212A, usbc:AMPHENOL_12402012E212A, symbol 12402012E212A:12402012E212A
- removed J4: VIN, Connector_PinHeader_2.54mm:PinHeader_1x02_P2.54mm_Vertical, symbol Connector:Conn_01x02_Pin
- removed J5: BAT, Connector_PinHeader_2.54mm:PinHeader_1x02_P2.54mm_Vertical, symbol Connector:Conn_01x02_Pin
- removed J6: DBG, Connector_PinHeader_2.54mm:PinHeader_1x03_P2.54mm_Vertical, symbol Connector:Conn_01x03_Pin
- removed J7: Conn_01x16_Pin, Connector_PinHeader_2.54mm:PinHeader_1x16_P2.54mm_Vertical, symbol Connector:Conn_01x16_Pin
- removed R11, R12, R13, R14, R16: 10K, Resistor_SMD:R_0805_2012Metric_Pad1.20x1.40mm_HandSolder, symbol Device:R
- removed R15, R17: 5.1k, Resistor_SMD:R_0805_2012Metric_Pad1.20x1.40mm_HandSolder, symbol Device:R
- removed U8: MCP7940N-xSN, Package_SO:SOIC-8_3.9x4.9mm_P1.27mm, symbol Timer_RTC:MCP7940N-xSN
- removed U9: RFM69HCW, RF_Module:HOPERF_RFM9XW_SMD, symbol RF_Module:RFM69HCW
- removed Y2: SC32S-7PF20PPM, sc32s:XTAL_SC32S-7PF20PPM_EPS, symbol Device:Crystal
Connections:
- no-connect marks 8 -> 0
Other:
- removed sheet Power
- added sheet CONNECTIONS (connections.kicad_sch)
- added sheet PERIPHERALS (peripherals.kicad_sch)
- added sheet POWER (power.kicad_sch)
- sheet MCU: file mcu.kicad_sch -> rp2040.kicad_sch
- note removed: "BATTERY"
- note removed: "DEBUG"
- note removed: "IO"
- note removed: "RADIO"
- note removed: "RTC"
- note removed: "SD CARD"
- note removed: "USB TYPE-C"
- note removed: "VIN"
