File: node_v4_0/node_v4_0/connections.kicad_sch (KiCad schematic)
At the start: 0 parts

Commit message: lots of stuff
Parts:
- added J4: Conn_02x08_Odd_Even, Connector_PinHeader_2.54mm:PinHeader_2x08_P2.54mm_Vertical, symbol Connector_Generic:Conn_02x08_Odd_Even
- added J5: Conn_02x02_Odd_Even, Connector_PinHeader_2.54mm:PinHeader_2x02_P2.54mm_Vertical, symbol Connector_Generic:Conn_02x02_Odd_Even
Connections:
- new net +3.3V: J4.1 (Pin_1), J4.2 (Pin_2), J5.2 (Pin_2)
- new net +5V: J4.4 (Pin_4)
- new net GND: J4.15 (Pin_15), J4.16 (Pin_16), J5.4 (Pin_4)
- new net GP6: J4.6 (Pin_6)
- new net GP7: J4.8 (Pin_8)
- new net GP8: J4.10 (Pin_10)
- new net MISO: J4.9 (Pin_9)
- new net MOSI: J4.7 (Pin_7)
- new net RX1: J4.5 (Pin_5)
- new net SCL: J4.14 (Pin_14)
- new net SDA: J4.12 (Pin_12)
- new net SPI_CK: J4.11 (Pin_11)
- new net SPI_CS: J4.13 (Pin_13)
- new net SWCLK: J5.1 (Pin_1)
- new net SWD: J5.3 (Pin_3)
- new net TX1: J4.3 (Pin_3)
