File: node_v4_0_sim/node_v4_0/peripherals.kicad_sch (KiCad schematic)
At the start: 23 parts, among them J3 Conn_Coaxial, U10 MCP7940N-xP, U11 SIM7080G, U6 RFM69HCW, U9 1042240820

Commit message: lots of stuff
Parts:
- U11: footprint Library:XCVR_SIM7080G -> WiSDOM:XCVR_SIM7080G
- XTAL1: footprint footprints:XTAL_SC32S-7PF20PPM_EPS -> WiSDOM:XTAL_SC32S-7PF20PPM_EPS
Connections:
- net RF_ANT: now reaches U11.32 (RF_ANT)
- net PWRKEY: now reaches U11.39 (PWRKEY)
- net GNSS_ANT: now reaches U11.68 (GNSS_ANT)
- no-connect marks 24 -> 41
Changed lines of the file:
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@@
 	)
 	(no_connect
+		(at 85.09 115.57)
+	)
+	(no_connect
 		(at 85.09 87.63)
 	)
@@
 	)
 	(no_connect
+		(at 43.18 73.66)
+	)
+	(no_connect
 		(at 153.67 124.46)
 	)
 	(no_connect
+		(at 85.09 113.03)
+	)
+	(no_connect
 		(at 85.09 100.33)
 	)
@@
 	)
 	(no_connect
+		(at 85.09 44.45)
+	)
+	(no_connect
+		(at 34.29 113.03)
+	)
+	(no_connect
 		(at 85.09 107.95)
 	)
@@
 	)
 	(no_connect
+		(at 85.09 49.53)
+	)
+	(no_connect
+		(at 34.29 110.49)
+	)
+	(no_connect
+		(at 34.29 87.63)
+	)
+	(no_connect
 		(at 153.67 137.16)
 	)
@@
 	)
 	(no_connect
+		(at 85.09 118.11)
+	)
+	(no_connect
 		(at 153.67 134.62)
 	)
 	(no_connect
+		(at 34.29 52.07)
+	)
+	(no_connect
 		(at 153.67 129.54)
 	)
 	(no_connect
+		(at 34.29 54.61)
+	)
+	(no_connect
+		(at 85.09 62.23)
+	)
+	(no_connect
 		(at 34.29 69.85)
 	)
 	(no_connect
+		(at 85.09 64.77)
+	)
+	(no_connect
+		(at 34.29 82.55)
+	)
+	(no_connect
 		(at 34.29 62.23)
 	)
 	(no_connect
+		(at 34.29 90.17)
+	)
+	(no_connect
+		(at 34.29 80.01)
+	)
+	(no_connect
 		(at 34.29 59.69)
 	)
 	(no_connect
+		(at 85.09 52.07)
+	)
+	(no_connect
 		(at 85.09 92.71)
 	)
@@
 	(wire
 		(pts
+			(xy 31.75 41.91) (xy 34.29 41.91)
+		)
+		(stroke
+			(width 0)
+			(type default)
+		)
+	)
+	(wire
+		(pts
 			(xy 256.54 27.94) (xy 256.54 30.48)
 		)
@@
 	(wire
 		(pts
+			(xy 85.09 57.15) (xy 87.63 57.15)
+		)
+		(stroke
+			(width 0)
+			(type default)
+		)
+	)
+	(wire
+		(pts
 			(xy 234.95 118.11) (xy 234.95 119.38)
 		)
@@
 	(wire
 		(pts
+			(xy 31.75 46.99) (xy 34.29 46.99)
+		)
+		(stroke
+			(width 0)
+			(type default)
+		)
+	)
+	(wire
+		(pts
 			(xy 91.44 146.05) (xy 91.44 148.59)
 		)
@@
 		)
 	)
+	(global_label "RF_ANT"
+		(shape input)
+		(at 87.63 57.15 0)
+		(fields_autoplaced yes)
+		(effects
+			(font
+				(size 1.27 1.27)
+			)
+			(justify left)
+		)
+		(property "Intersheetrefs" "${INTERSHEET_REFS}"
+			(at 97.3281 57.15 0)
+			(effects
+				(font
+					(size 1.27 1.27)
+				)
+				(justify left)
+				(hide yes)
+			)
+		)
+	)
 	(global_label "SPI_CK"
 		(shape input)
@@
 		)
 	)
+	(global_label "PWRKEY"
+		(shape input)
+		(at 31.75 41.91 180)
+		(fields_autoplaced yes)
+		(effects
+			(font
+				(size 1.27 1.27)
+			)
+			(justify right)
+		)
+		(property "Intersheetrefs" "${INTERSHEET_REFS}"
+			(at 21.2658 41.91 0)
+			(effects
+				(font
+					(size 1.27 1.27)
+				)
+				(justify right)
+				(hide yes)
+			)
+		)
+	)
 	(global_label "RX1"
 		(shape input)
@@
 		)
 	)
+	(global_label "GNSS_ANT"
+		(shape input)
+		(at 31.75 46.99 180)
+		(fields_autoplaced yes)
+		(effects
+			(font
+				(size 1.27 1.27)
+			)
+			(justify right)
+		)
+		(property "Intersheetrefs" "${INTERSHEET_REFS}"
+			(at 19.391 46.99 0)
+			(effects
+				(font
+					(size 1.27 1.27)
+				)
+				(justify right)
+				(hide yes)
+			)
+		)
+	)
 	(global_label "MISO"
 		(shape input)
@@
 			)
 		)
-		(property "Footprint" "Library:XCVR_SIM7080G"
+		(property "Footprint" "WiSDOM:XCVR_SIM7080G"
 			(at 59.69 77.47 0)
 			(effects
@@
 			)
 		)
-		(property "Footprint" "footprints:XTAL_SC32S-7PF20PPM_EPS"
+		(property "Footprint" "WiSDOM:XTAL_SC32S-7PF20PPM_EPS"
 			(at 245.11 123.19 0)
 			(effects
