File: node_v4_0_sim/node_v4_0/power.kicad_sch (KiCad schematic)
At the start: 23 parts, among them J1 Conn_01x02_Pin, J2 12402012E212A, Q1 DMG2301L, U3 AP2112K-3.3, U4 CAT3200-5, U5 MCP73831-2-OT

Commit message: lots of stuff
Parts:
- J2: footprint usbc:AMPHENOL_12402012E212A -> WiSDOM:AMPHENOL_12402012E212A
Changed lines of the file:
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@@
 			)
 		)
-		(property "Footprint" "usbc:AMPHENOL_12402012E212A"
+		(property "Footprint" "WiSDOM:AMPHENOL_12402012E212A"
 			(at 91.186 130.556 0)
 			(effects
