File: node_v4_0_sim/node_v4_0/rp2040.kicad_sch (KiCad schematic)
At the start: 29 parts, among them U1 RP2040, U2 W25Q128JVS, U7 PTS526 SK15 SMTR2 LFS, U8 PTS526 SK15 SMTR2 LFS

Commit message: lots of stuff
Parts:
- U1: footprint RP2040_minimal_r2:RP2040-QFN-56 -> Package_DFN_QFN:QFN-56-1EP_7x7mm_P0.4mm_EP3.2x3.2mm
- U7, U8: footprint pts526:SMT_FS -> WiSDOM:PTS526
- X1: footprint custom:XTAL-445 -> WiSDOM:XTAL-445
Connections:
- net CS: no longer U8.1, U8.2
- net PWRKEY: now reaches U1.17 (GPIO14)
- new net: R10.1, U8.1, U8.2
- now unconnected: U8.3, U8.4
Other:
- moved on the sheet: U8
Changed lines of the file:
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@@
 	)
 	(junction
+		(at 240.03 111.76)
+		(diameter 0)
+		(color 0 0 0 0)
+	)
+	(junction
+		(at 240.03 114.3)
+		(diameter 0)
+		(color 0 0 0 0)
+	)
+	(junction
 		(at 76.2 76.2)
 		(diameter 0)
@@
 	(wire
 		(pts
+			(xy 95.25 135.89) (xy 97.79 135.89)
+		)
+		(stroke
+			(width 0)
+			(type default)
+		)
+	)
+	(wire
+		(pts
 			(xy 67.31 76.2) (xy 69.85 76.2)
 		)
@@
 	(wire
 		(pts
+			(xy 240.03 114.3) (xy 242.57 114.3)
+		)
+		(stroke
+			(width 0)
+			(type default)
+		)
+	)
+	(wire
+		(pts
 			(xy 139.7 35.56) (xy 152.4 35.56)
 		)
@@
 	(wire
 		(pts
-			(xy 238.76 114.3) (xy 242.57 114.3)
+			(xy 238.76 114.3) (xy 240.03 114.3)
 		)
 		(stroke
@@
 	(wire
 		(pts
+			(xy 240.03 111.76) (xy 242.57 111.76)
+		)
+		(stroke
+			(width 0)
+			(type default)
+		)
+	)
+	(wire
+		(pts
 			(xy 26.67 101.6) (xy 31.75 101.6)
 		)
@@
 	(wire
 		(pts
-			(xy 238.76 111.76) (xy 242.57 111.76)
+			(xy 238.76 111.76) (xy 240.03 111.76)
 		)
 		(stroke
@@
 		)
 	)
+	(global_label "PWRKEY"
+		(shape input)
+		(at 97.79 135.89 0)
+		(fields_autoplaced yes)
+		(effects
+			(font
+				(size 1.27 1.27)
+			)
+			(justify left)
+		)
+		(property "Intersheetrefs" "${INTERSHEET_REFS}"
+			(at 108.2742 135.89 0)
+			(effects
+				(font
+					(size 1.27 1.27)
+				)
+				(justify left)
+				(hide yes)
+			)
+		)
+	)
 	(global_label "SWCLK"
 		(shape input)
@@
 			)
 		)
-		(property "Footprint" "RP2040_minimal_r2:RP2040-QFN-56"
+		(property "Footprint" "Package_DFN_QFN:QFN-56-1EP_7x7mm_P0.4mm_EP3.2x3.2mm"
 			(at 44.45 133.35 0)
 			(effects
@@
 			)
 		)
-		(property "Footprint" "custom:XTAL-445"
+		(property "Footprint" "WiSDOM:XTAL-445"
 			(at 171.45 74.93 0)
 			(effects
@@
 			)
 		)
-		(property "Footprint" "pts526:SMT_FS"
+		(property "Footprint" "WiSDOM:PTS526"
 			(at 233.68 85.852 0)
 			(effects
@@
 		(lib_id "2024-05-28_14-35-54:PTS526_SK15_SMTR2_LFS")
 		(at 233.68 111.76 0)
+		(mirror y)
 		(unit 1)
 		(exclude_from_sim no)
@@
 		(on_board yes)
 		(dnp no)
-		(fields_autoplaced yes)
 		(property "Reference" "U8"
-			(at 233.045 105.41 0)
+			(at 234.315 105.41 0)
 			(effects
 				(font
@@
 		)
 		(property "Value" "PTS526 SK15 SMTR2 LFS"
-			(at 233.045 107.95 0)
+			(at 234.315 107.95 0)
 			(effects
 				(font
@@
 			)
 		)
-		(property "Footprint" "pts526:SMT_FS"
-			(at 232.41 106.172 0)
+		(property "Footprint" "WiSDOM:PTS526"
+			(at 234.95 106.172 0)
 			(effects
 				(font
@@
 		)
 		(property "Datasheet" "PTS526 SK15 SMTR2 LFS"
-			(at 233.426 107.95 0)
+			(at 233.934 107.95 0)
 			(effects
 				(font
