File: node_v4_0_sim/node_v4_0/node_v4_0.kicad_pcb (KiCad board)
At the start: 4 copper layers, 45.7 x 76.2 mm, 86 parts, among them J1 Conn_01x02_Pin, J2 12402012E212A, J3 Conn_Coaxial, J4 Conn_01x16_Pin, J5 Conn_02x02_Odd_Even, J6 GNSS_ANT, J7 RF_ANT, Q1 DMG2301L, U1 RP2040, U10 MCP7940N-xP, U11 SIM7080G, U2 W25Q128JVS, U3 AP2112K-3.3, U4 CAT3200-5, U5 MCP73831-2-OT, U6 RFM69HCW, U7 PTS526 SK15 SMTR2 LFS, U8 PTS526 SK15 SMTR2 LFS, U9 1042240820

Commit message: placed everything in the sim version
Parts:
- moved R11 133.6 mm to (165.4, 117.1), turned to -90 degrees
- moved C42 127.6 mm to (164.5, 88.7), turned to 90 degrees
- moved R12 119.4 mm to (149.4, 123.2)
- moved R13 117.7 mm to (149.4, 120.9)
- moved C29 111.4 mm to (139.7, 110.5)
- moved C34 100.4 mm to (165.1, 114.1), turned to 90 degrees
- moved C35 96.2 mm to (162.8, 111.5)
- moved L1 92.9 mm to (168.7, 110.0), turned to 180 degrees
- moved R14 91.4 mm to (163.3, 82.5)
- moved C36 87.0 mm to (146.1, 123.2), turned to 180 degrees
- moved C38 85.1 mm to (160.0, 89.5), turned to 90 degrees
- moved C37 84.5 mm to (146.1, 120.9), turned to 180 degrees
- moved C28 77.8 mm to (139.5, 108.7)
- moved C40 75.2 mm to (156.4, 89.2), turned to 180 degrees
- moved C39 75.2 mm to (156.5, 85.9), turned to 180 degrees
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Routing:
- net +1V1: track 17.5 -> 64.6 mm, vias 0 -> 3
- net Net-(J2-CC1_B): track 0.00 -> 3.75 mm
- net Net-(J2-CC1_A): track 0.00 -> 3.23 mm
- net USB+: track 9.38 -> 12.4 mm, vias 0 -> 2
- net USB-: track 9.21 -> 11.5 mm, vias 0 -> 2
- net Net-(U1-USB_DP): track 9.54 -> 10.9 mm
- net +3.3V: track 50.1 -> 51.1 mm
- net GND: vias 2 -> 30
