File: node-rp2040/node_v6_0_0/peripherals.kicad_sch (KiCad schematic)
At the start: 30 parts, among them U11 1042240820, U12 CAT24M01W, U6 RFM69HCW, U7 PCF8523T, U8 SP3485EN, U9 SIM7080G

Commit message: i should have made this more than one commit but: 1) started poking around in v5 to find and solve a sim card problem, forgot about it and moved on 2) created v6, modified the schematic somewhat, removed some parts, began laying out the pcb again this time as a 6 layer board 3) fixed the library setup so now it uses symbols and footprints from the packages available alongside kicad (in void linux at least) for all standard stuff PLUS the wisdom libraries and the jlcpcb prefered parts library
Parts:
- C17, C28, C30, C34, C35, C36, C37, C38, C44: footprint JLCPCB-Kicad-Footprints:C_0402 -> JLCPCB:C_0402
- C18, C29, C31, C41, C42, C45: footprint JLCPCB-Kicad-Footprints:C_0805 -> JLCPCB:C_0805
- C32, C33: footprint JLCPCB-Kicad-Footprints:C_0603 -> JLCPCB:C_0603
- R11, R12, R13: footprint JLCPCB-Kicad-Footprints:R_0402 -> JLCPCB:R_0402
- U8: footprint JLCPCB-Kicad-Footprints:SOIC-8_L5.0-W4.0-P1.27-LS6.0-BL -> JLCPCB:SOIC-8_L5.0-W4.0-P1.27-LS6.0-BL
Changed lines of the file:
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@@
 			)
 		)
-		(property "Footprint" "JLCPCB-Kicad-Footprints:C_0402"
+		(property "Footprint" "JLCPCB:C_0402"
 			(at 112.522 35.56 90)
 			(effects
@@
 			)
 		)
-		(property "Footprint" "JLCPCB-Kicad-Footprints:R_0402"
+		(property "Footprint" "JLCPCB:R_0402"
 			(at 193.04 32.258 90)
 			(effects
@@
 			)
 		)
-		(property "Footprint" "JLCPCB-Kicad-Footprints:C_0805"
+		(property "Footprint" "JLCPCB:C_0805"
 			(at 164.592 149.86 90)
 			(effects
@@
 			)
 		)
-		(property "Footprint" "JLCPCB-Kicad-Footprints:SOIC-8_L5.0-W4.0-P1.27-LS6.0-BL"
+		(property "Footprint" "JLCPCB:SOIC-8_L5.0-W4.0-P1.27-LS6.0-BL"
 			(at 247.65 163.83 0)
 			(effects
@@
 			)
 		)
-		(property "Footprint" "JLCPCB-Kicad-Footprints:C_0402"
+		(property "Footprint" "JLCPCB:C_0402"
 			(at 160.782 82.55 90)
 			(effects
@@
 			)
 		)
-		(property "Footprint" "JLCPCB-Kicad-Footprints:C_0805"
+		(property "Footprint" "JLCPCB:C_0805"
 			(at 214.122 149.86 90)
 			(effects
@@
 			)
 		)
-		(property "Footprint" "JLCPCB-Kicad-Footprints:C_0805"
+		(property "Footprint" "JLCPCB:C_0805"
 			(at 267.462 114.3 90)
 			(effects
@@
 			)
 		)
-		(property "Footprint" "JLCPCB-Kicad-Footprints:C_0402"
+		(property "Footprint" "JLCPCB:C_0402"
 			(at 169.672 41.91 90)
 			(effects
@@
 			)
 		)
-		(property "Footprint" "JLCPCB-Kicad-Footprints:C_0402"
+		(property "Footprint" "JLCPCB:C_0402"
 			(at 266.192 33.02 90)
 			(effects
@@
 			)
 		)
-		(property "Footprint" "JLCPCB-Kicad-Footprints:C_0805"
+		(property "Footprint" "JLCPCB:C_0805"
 			(at 125.222 35.56 90)
 			(effects
@@
 			)
 		)
-		(property "Footprint" "JLCPCB-Kicad-Footprints:C_0805"
+		(property "Footprint" "JLCPCB:C_0805"
 			(at 172.212 82.55 90)
 			(effects
@@
 			)
 		)
-		(property "Footprint" "JLCPCB-Kicad-Footprints:C_0603"
+		(property "Footprint" "JLCPCB:C_0603"
 			(at 267.97 99.568 90)
 			(effects
@@
 			)
 		)
-		(property "Footprint" "JLCPCB-Kicad-Footprints:C_0805"
+		(property "Footprint" "JLCPCB:C_0805"
 			(at 136.652 35.56 90)
 			(effects
@@
 			)
 		)
-		(property "Footprint" "JLCPCB-Kicad-Footprints:C_0402"
+		(property "Footprint" "JLCPCB:C_0402"
 			(at 256.032 114.3 90)
 			(effects
@@
 			)
 		)
-		(property "Footprint" "JLCPCB-Kicad-Footprints:C_0402"
+		(property "Footprint" "JLCPCB:C_0402"
 			(at 202.692 149.86 90)
 			(effects
@@
 			)
 		)
-		(property "Footprint" "JLCPCB-Kicad-Footprints:C_0402"
+		(property "Footprint" "JLCPCB:C_0402"
 			(at 153.162 149.86 90)
 			(effects
@@
 			)
 		)
-		(property "Footprint" "JLCPCB-Kicad-Footprints:R_0402"
+		(property "Footprint" "JLCPCB:R_0402"
 			(at 193.04 34.798 90)
 			(effects
@@
 			)
 		)
-		(property "Footprint" "JLCPCB-Kicad-Footprints:C_0603"
+		(property "Footprint" "JLCPCB:C_0603"
 			(at 267.97 86.868 90)
 			(effects
@@
 			)
 		)
-		(property "Footprint" "JLCPCB-Kicad-Footprints:C_0402"
+		(property "Footprint" "JLCPCB:C_0402"
 			(at 179.832 41.91 90)
 			(effects
@@
 			)
 		)
-		(property "Footprint" "JLCPCB-Kicad-Footprints:R_0402"
+		(property "Footprint" "JLCPCB:R_0402"
 			(at 233.68 48.768 90)
 			(effects
@@
 			)
 		)
-		(property "Footprint" "JLCPCB-Kicad-Footprints:C_0402"
+		(property "Footprint" "JLCPCB:C_0402"
 			(at 216.662 52.07 90)
 			(effects
