File: node-rp2040/node_v6_2_0/connections.kicad_sch (KiCad schematic)
At the start: 15 parts, among them J11 Barrel_Jack_Switch, J2 U.FL, J3 Conn_Coaxial, J4 Conn_01x10, J5 Conn_01x10, J6 U.FL, J7 Barrel_Jack_Switch, J9 U.FL

Commit message: finished layout v6.2
Parts:
- C43: now fitted; now in the parts list
Changed lines of the file:
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@@
 		(unit 1)
 		(exclude_from_sim no)
-		(in_bom no)
+		(in_bom yes)
 		(on_board yes)
-		(dnp yes)
+		(dnp no)
 		(property "Reference" "C43"
 			(at 190.5 72.39 90)
